Commit message: added sym_type parameter in transmission

File: pal_pro_gripper_description/urdf/gripper.ros2_control.xacro (robot description, xacro)
@@ -45,5 +45,5 @@
     joint-->
     <xacro:include filename="$(find pal_pro_gripper_description)/urdf/gripper.transmission.xacro" />
-    <xacro:pal_pro_gripper_transmission name="${name}_finger"/>
+    <xacro:pal_pro_gripper_transmission name="${name}_finger" sim_type="${sim_type}"/>
   </xacro:macro>
 </robot>

File: pal_pro_gripper_description/urdf/gripper.transmission.xacro (robot description, xacro)
@@ -13,5 +13,5 @@
  -->
 <robot xmlns:xacro="http://ros.org/wiki/xacro">
-  <xacro:macro name="pal_pro_gripper_transmission" params="name">
+  <xacro:macro name="pal_pro_gripper_transmission" params="name sim_type:=gazebo">
     <transmission name="${name}_trans">
         <plugin>pal_pro_gripper_transmissions/PalGripperTransmission</plugin>

Commit message: fixed param

File: pal_pro_gripper_description/urdf/gripper.ros2_control.xacro (robot description, xacro)
@@ -13,6 +13,6 @@
 -->
 <robot xmlns:xacro="http://ros.org/wiki/xacro">
-  <xacro:macro name="ros2_control_pal_pro_gripper" params="name reduction">
-    <xacro:macro name="ros2_control_pal_pro_gripper_mimic_joint" params="mimic_joint_name actuated_joint_name multipliers sim_type:=gazebo">
+  <xacro:macro name="ros2_control_pal_pro_gripper" params="name reduction sim_type:=gazebo">
+    <xacro:macro name="ros2_control_pal_pro_gripper_mimic_joint" params="mimic_joint_name actuated_joint_name multipliers ">
       <joint name="${mimic_joint_name}">
         <param name="mimic">${actuated_joint_name}</param>

Commit message: fixed multiplier arg

File: pal_pro_gripper_description/urdf/gripper.ros2_control.xacro (robot description, xacro)
@@ -14,5 +14,5 @@
 <robot xmlns:xacro="http://ros.org/wiki/xacro">
   <xacro:macro name="ros2_control_pal_pro_gripper" params="name reduction sim_type:=gazebo">
-    <xacro:macro name="ros2_control_pal_pro_gripper_mimic_joint" params="mimic_joint_name actuated_joint_name multipliers ">
+    <xacro:macro name="ros2_control_pal_pro_gripper_mimic_joint" params="mimic_joint_name actuated_joint_name multiplier ">
       <joint name="${mimic_joint_name}">
         <param name="mimic">${actuated_joint_name}</param>

Commit message: Change the init value + change the lower limit temporally

File: pal_pro_gripper_description/urdf/gripper.ros2_control.xacro (robot description, xacro)
@@ -23,5 +23,12 @@
       <command_interface name="position"/>
       <state_interface name="position">
-        <param name="initial_value">0.07938</param>
+        <!-- TODO: set initial_value back to 0.07938 when moving to Gazebo Harmonic or ROS 2 Jazzy -->
+        <!-- See https://robotics.stackexchange.com/questions/85506/how-to-do-mimic-joints-that-work-in-gazebo for more information -->
+        <xacro:if value="${gazebo_version == 'classic'}">
+          <param name="initial_value">0.07938</param>
+        </xacro:if>
+        <xacro:if value="${gazebo_version == 'gazebo'}">
+          <param name="initial_value">0.0</param>
+        </xacro:if>
       </state_interface>
       <state_interface name="velocity"/>

File: pal_pro_gripper_description/urdf/gripper.urdf.xacro (robot description, xacro)
@@ -8,4 +8,12 @@
     </link>
     <xacro:property name="finger_joint_name" value="${name + '_finger_joint' if side == 'left' else name + '_finger_' + side + '_joint'}" />
+    <!-- TODO: set lower limit back to 0 when moving to Gazebo Harmonic or ROS 2 Jazzy -->
+    <!-- See https://github.com/gazebosim/gz-sim/issues/1684 for more information -->
+    <xacro:if value="${gazebo_version == 'classic'}">
+      <xacro:property name="gripper_lower_limit" value="0.0"/>
+    </xacro:if>
+    <xacro:if value="${gazebo_version == 'gazebo'}">
+      <xacro:property name="gripper_lower_limit" value="-1e-3"/>
+    </xacro:if>
     <joint name="${finger_joint_name}" type="prismatic">
       <xacro:origin_finger_joint reflect="${reflect}"/>
@@ -13,6 +21,6 @@
       <child link="${name}_screw_${side}_link"/>
       <axis xyz="0 1 0"/>
-      <limit lower="0.0" upper="0.07938" velocity="2" effort="10.0"/>
-      <safety_controller k_position="20" k_velocity="20" soft_lower_limit="${0.0 + gripper_eps}" soft_upper_limit="${0.07938 - gripper_eps}" />
+      <limit lower="${gripper_lower_limit}" upper="0.07938" velocity="2" effort="10.0"/>
+      <safety_controller k_position="20" k_velocity="20" soft_lower_limit="${gripper_lower_limit + gripper_eps}" soft_upper_limit="${0.07938 - gripper_eps}" />
       <xacro:if value="${side == 'left'}">
         <dynamics damping="0.03"/>
