Commit message: Add safety controller

File: pal_pro_gripper_description/urdf/gripper.urdf.xacro (robot description, xacro)
@@ -14,4 +14,5 @@
       <axis xyz="0 1 0"/>
       <limit lower="0.0" upper="0.07938" velocity="2" effort="0.1"/>
+      <safety_controller k_position="20" k_velocity="20" soft_lower_limit="${0.0 + gripper_eps}" soft_upper_limit="${0.07938 - gripper_eps}" />
       <xacro:if value="${side == 'left'}">
         <dynamics damping="0.03"/>
@@ -132,4 +133,6 @@
     <xacro:property name="gripper_base_type" value="${'base_link_tc' if tool_changer else 'base_link_ntc'}" />
     <xacro:property name="finger_offset" value="${0.0 if tool_changer else 0.006}" />
+    <!--Constant parameters-->
+    <xacro:property name="gripper_eps" value="0.0" />
     <!-- Properties files -->
     <xacro:include filename="$(find pal_pro_gripper_description)/urdf/gripper.properties.xacro"/>

Commit message: Reduce the gripper opening position to avoid hit the joint limit when completely open

File: pal_pro_gripper_description/urdf/gripper.urdf.xacro (robot description, xacro)
@@ -21,6 +21,6 @@
       <child link="${name}_screw_${side}_link"/>
       <axis xyz="0 1 0"/>
-      <limit lower="${gripper_lower_limit}" upper="0.07938" velocity="2" effort="10.0"/>
-      <safety_controller k_position="20" k_velocity="20" soft_lower_limit="${gripper_lower_limit + gripper_eps}" soft_upper_limit="${0.07938 - gripper_eps}" />
+      <limit lower="${gripper_lower_limit}" upper="0.07" velocity="2" effort="10.0"/>
+      <safety_controller k_position="20" k_velocity="20" soft_lower_limit="${gripper_lower_limit + gripper_eps}" soft_upper_limit="${0.07 - gripper_eps}" />
       <xacro:if value="${side == 'left'}">
         <dynamics damping="0.03"/>
