Commit message: adapt transmission for the mujoco ros2 control

File: pal_pro_gripper_description/urdf/gripper.transmission.xacro (robot description, xacro)
@@ -13,12 +13,11 @@
  -->
 <robot xmlns:xacro="http://ros.org/wiki/xacro">
-  <xacro:macro name="pal_pro_gripper_transmission" params="name sim_type:=gazebo">
+  <xacro:macro name="pal_pro_gripper_transmission" params="name sim_type:=^|gazebo">
     <transmission name="${name}_trans">
         <plugin>pal_pro_gripper_transmissions/PalGripperTransmission</plugin>
-        <!-- <actuator name="${name}_actuator" role="actuator1"/>  -->
-        <xacro:if value="${sim_type == 'mujoco' or sim_type == 'mujoco-ros2-control'}">
+        <xacro:if value="${sim_type == 'mujoco-ros2-control'}">
           <actuator name="${name}_joint" role="actuator1"/>
         </xacro:if>
-        <xacro:unless value="${sim_type == 'mujoco' or sim_type == 'mujoco-ros2-control'}">
+        <xacro:unless value="${sim_type == 'mujoco-ros2-control'}">
           <actuator name="${name}_actuator" role="actuator1"/>
         </xacro:unless>
