Commit message: added sim_type for transmission

File: pal_pro_gripper_description/ros2_control/ros2_control.urdf.xacro (robot description, xacro)
@@ -37,5 +37,5 @@
       </hardware>
       <!-- pal-pro-gripper -->
-      <xacro:ros2_control_pal_pro_gripper name="gripper" reduction="1.0"/>
+      <xacro:ros2_control_pal_pro_gripper name="gripper" reduction="1.0" sim_type="${sim_type}"/>
     </ros2_control>
   </xacro:macro>

File: pal_pro_gripper_description/urdf/gripper.ros2_control.xacro (robot description, xacro)
@@ -14,5 +14,5 @@
 <robot xmlns:xacro="http://ros.org/wiki/xacro">
   <xacro:macro name="ros2_control_pal_pro_gripper" params="name reduction">
-    <xacro:macro name="ros2_control_pal_pro_gripper_mimic_joint" params="mimic_joint_name actuated_joint_name multiplier">
+    <xacro:macro name="ros2_control_pal_pro_gripper_mimic_joint" params="mimic_joint_name actuated_joint_name multipliers sim_type:=gazebo">
       <joint name="${mimic_joint_name}">
         <param name="mimic">${actuated_joint_name}</param>

Commit message: Add support for new gazebo

File: pal_pro_gripper_description/ros2_control/ros2_control.urdf.xacro (robot description, xacro)
@@ -22,5 +22,10 @@
           </xacro:if>
           <xacro:if value="${sim_type == 'gazebo'}">
-            <plugin>gazebo_ros2_control/GazeboSystem</plugin>
+            <xacro:if value="${gazebo_version == 'classic'}">
+              <plugin>gazebo_ros2_control/GazeboSystem</plugin>
+            </xacro:if>
+            <xacro:if value="${gazebo_version == 'gazebo'}">
+              <plugin>gz_ros2_control/GazeboSimSystem</plugin>
+            </xacro:if>
           </xacro:if>
         </xacro:if>

File: pal_pro_gripper_description/urdf/gripper.ros2_control.xacro (robot description, xacro)
@@ -14,8 +14,19 @@
 <robot xmlns:xacro="http://ros.org/wiki/xacro">
   <xacro:macro name="ros2_control_pal_pro_gripper" params="name reduction sim_type:=no-simulation">
+    <hardware>
+      <xacro:if value="${gazebo_version == 'classic'}">
+        <plugin>gazebo_ros2_control/GazeboSystem</plugin>
+      </xacro:if>
+      <xacro:if value="${gazebo_version == 'gazebo'}">
+        <plugin>gz_ros2_control/GazeboSimSystem</plugin>
+      </xacro:if>
+    </hardware>
     <xacro:macro name="ros2_control_pal_pro_gripper_mimic_joint" params="mimic_joint_name actuated_joint_name multiplier sim_type:=no-simulation">
       <joint name="${mimic_joint_name}">
         <param name="mimic">${actuated_joint_name}</param>
         <param name="multiplier">${multiplier}</param>
+        <state_interface name="position"/>
+        <state_interface name="velocity"/>
+        <state_interface name="effort"/>
       </joint>
     </xacro:macro>

File: pal_pro_gripper_description/urdf/gripper.urdf.xacro (robot description, xacro)
@@ -13,5 +13,5 @@
       <child link="${name}_screw_${side}_link"/>
       <axis xyz="0 1 0"/>
-      <limit lower="0.0" upper="0.07938" velocity="2" effort="0.1"/>
+      <limit lower="0.0" upper="0.07938" velocity="2" effort="10.0"/>
       <safety_controller k_position="20" k_velocity="20" soft_lower_limit="${0.0 + gripper_eps}" soft_upper_limit="${0.07938 - gripper_eps}" />
       <xacro:if value="${side == 'left'}">
@@ -274,12 +274,14 @@
       <mu2>0.9</mu2>
     </gazebo>
-    <gazebo>
-      <plugin name="mimic_joint_plugin_right" filename="libgazebo_ros_mimic_joint.so">
-        <joint>gripper_finger_joint</joint>
-        <mimicJoint>gripper_finger_right_joint</mimicJoint>
-        <multiplier>1.0</multiplier>
-        <offset>0.0</offset>
-      </plugin>
-    </gazebo>
+    <xacro:if value="${gazebo_version == 'classic'}">
+      <gazebo>
+        <plugin name="mimic_joint_plugin_right" filename="libgazebo_ros_mimic_joint.so">
+          <joint>gripper_finger_joint</joint>
+          <mimicJoint>gripper_finger_right_joint</mimicJoint>
+          <multiplier>1.0</multiplier>
+          <offset>0.0</offset>
+        </plugin>
+      </gazebo>
+    </xacro:if>
     <!-- Base finger links -->
     <gazebo reference="${name}_base_finger_left_link">
