Commit message: add check for the value of the sim_type arg

File: pal_pro_gripper_description/robots/pal_pro_gripper.urdf.xacro (robot description, xacro)
@@ -9,8 +9,9 @@
     <!-- false, true -->
     <xacro:arg name="use_sim_time" default="False"/>
-    <!-- mujoco-ros2-control, mujoco, gazebo, no-simulation -->
+    <!-- mujoco-ros2-control, mujoco, gazebo-->
     <xacro:arg name="sim_type" default="gazebo" />
     <!-- false, position, motor -->
-    <xacro:arg name="mj_control" default="position" />
+    <xacro:arg name="mj_control" default="false" />
+    <!-- floor -->
     <xacro:arg name="world_name" default="floor" />
     <!-- PROPERTIES -->
@@ -23,4 +24,11 @@
     <xacro:property name="mj_control" value="$(arg mj_control)"/>
     <xacro:property name="world_name" value="$(arg world_name)"/>
+    <!-- Properties check -->
+    <xacro:if value="${sim_type not in ['mujoco-ros2-control', 'mujoco', 'gazebo']}">
+        <xacro:wrong_sim_type />
+    </xacro:if>
+    <xacro:unless value="$(arg use_sim_time)">
+        <xacro:property name="sim_type" value="gazebo" />
+    </xacro:unless>
     <!-- INCLUDES -->
     <!-- Helpers -->

Commit message: move mj tags to gripper.urdf.xacro

File: pal_pro_gripper_description/robots/pal_pro_gripper.urdf.xacro (robot description, xacro)
@@ -47,57 +47,6 @@
     </xacro:pal_pro_gripper>
     <!-- MUJOCO -->
-    <xacro:if value="${sim_type == 'mujoco' or sim_type == 'mujoco-ros2-control'}">
-        <!-- Mujoco Includes -->
-        <xacro:include filename="$(find pal_pro_gripper_description)/mujoco/mj_tags.xacro" />
-        <xacro:include filename="$(find pal_mujoco_scenes)/scenes/${world_name}.xacro" />
-        <mujoco_inputs>
-            <!-- Mujoco environment -->
-            <scene>
-                <xacro:mj_scene/>
-            </scene>
-            <raw_inputs>
-                <!-- Contact-->
-                <xacro:mj_gripper_contact name="gripper"/>
-                <!-- Equality-->
-                <xacro:mj_gripper_equality name="gripper" anchor_r="0.014 -0.0015 0" anchor_l="0.014 -0.001 0"/>
-                <!-- Actuator-->
-                <actuator>
-                    <xacro:mj_gripper_actuators name="gripper"/>
-                </actuator>
-                <default>
-                    <default class="visual">
-                        <geom group="2" type="mesh" contype="0" conaffinity="0"/>
-                    </default>
-                    <default class="collision">
-                        <geom group="3" type="mesh"/>
-                    </default>
-                </default>
-            </raw_inputs>
-            <processed_inputs>
-                <!-- Specifying decompose_mesh will set the `decompose` flag when using obj2mjcf -->
-                <!-- <decompose_mesh mesh_name="arm2_link" threshold="0.05"/>
-                <decompose_mesh mesh_name="arm3_link" threshold="0.05"/> -->
-                <!-- <decompose_mesh mesh_name="arm4_link" threshold="0.05"/> -->
-                <!-- The camera with the specified values will be added at the specified site name. -->
-                <!-- The position and quaterinion will be filled in by the converter -->
-                <!-- <camera site="pelvis_1_link" name="camera" fovy="58" mode="fixed" resolution="640 480" pos="2 2 2" quat="1 0 0 0"/> -->
-                <!-- Adds a lidar tag below a site tag to support a lidar sensor. -->
-                <!-- In the URDF, we assume that that the sensor frame has the Z-axis pointed directly up in the sensor -->
-                <!-- frame. This tag will create rangefinders in the MJCF between min_angle and max_angle at each -->
-                <!-- angle_increment rotated about the replicate frame's Y axis. The hardware intercface then combines -->
-                <!-- them into a single LaserScan message. -->
-                <!-- <lidar ref_site="torso_link" sensor_name="rf" min_angle="-0.3" max_angle="0.3" angle_increment="0.025" /> -->
-                <!-- The element with the type and name as listed below will be modified with the remaining attributes -->
-                <!-- If the attribute already existed, it will be overwritten -->
-                <!-- Note that the type and name elements are required -->
-                <modify_element type="joint" name="gripper_outer_finger_left_joint" actuatorfrcrange="-8 8"/>
-                <modify_element type="joint" name="gripper_outer_finger_right_joint" actuatorfrcrange="-8 8"/>
-                <modify_element type="joint" name="gripper_inner_finger_left_joint" actuatorfrcrange="-8 8"/>
-                <modify_element type="joint" name="gripper_finger_right_joint" actuatorfrcrange="-8 8"/>
-                <modify_element type="joint" name="gripper_fingertip_left_joint" actuatorfrcrange="-8 8"/>
-                <modify_element type="joint" name="gripper_fingertip_right_joint" actuatorfrcrange="-8 8"/>
-                <modify_element type="joint" name="gripper_finger_joint" actuatorfrcrange="-8 8" damping="1.5"/>
-            </processed_inputs>
-        </mujoco_inputs>
+    <xacro:if value="${sim_type in ['mujoco', 'mujoco-ros2-control']}">
+        <xacro:pal_pro_gripper_mj world_name="${world_name}" mj_control="${mj_control}"/>
     </xacro:if>
     <!-- ROS 2 Control -->

File: pal_pro_gripper_description/urdf/gripper.urdf.xacro (robot description, xacro)
@@ -304,3 +304,54 @@
     </gazebo>
   </xacro:macro>
+  <xacro:macro name="pal_pro_gripper_mj" params="mj_control world_name">
+    <xacro:include filename="$(find pal_pro_gripper_description)/mujoco/mj_tags.xacro" />
+    <xacro:include filename="$(find pal_mujoco_scenes)/scenes/${world_name}.xacro" />
+    <mujoco_inputs>
+      <!-- Mujoco environment -->
+      <scene>
+          <xacro:mj_scene/>
+      </scene>
+      <raw_inputs>
+        <!-- Contact-->
+        <xacro:mj_gripper_contact name="gripper"/>
+        <!-- Equality-->
+        <xacro:mj_gripper_equality name="gripper" anchor_r="0.014 -0.0015 0" anchor_l="0.014 -0.001 0"/>
+        <!-- Actuator-->
+        <actuator>
+            <xacro:mj_gripper_actuators name="gripper"/>
+        </actuator>
+        <default>
+            <default class="visual">
+                <geom group="2" type="mesh" contype="0" conaffinity="0"/>
+            </default>
+            <default class="collision">
+                <geom group="3" type="mesh"/>
+            </default>
+        </default>
+      </raw_inputs>
+      <processed_inputs>
+        <!-- Specifying decompose_mesh will set the `decompose` flag when using obj2mjcf -->
+        <!-- <decompose_mesh mesh_name="{mesh_name}" threshold=" {threshold_value}"/> -->
+        <!-- The camera with the specified values will be added at the specified site name. -->
+        <!-- The position and quaterinion will be filled in by the converter -->
+        <!-- <camera site="{site_name}" name="{camera_name}" fovy="{fovy_value}" mode="{mode_type}" resolution="{resolution_values}"/> -->
+        <!-- Adds a lidar tag below a site tag to support a lidar sensor. -->
+        <!-- In the URDF, we assume that that the sensor frame has the Z-axis pointed directly up in the sensor -->
+        <!-- frame. This tag will create rangefinders in the MJCF between min_angle and max_angle at each -->
+        <!-- angle_increment rotated about the replicate frame's Y axis. The hardware intercface then combines -->
+        <!-- them into a single LaserScan message. -->
+        <!-- <lidar ref_site="{link_name}" sensor_name="{sensor_name}" min_angle="{min_angle_value}" max_angle="{max_angle_value}" angle_increment="{angle_increment_value}" /> -->
+          <!-- The element with the type and name as listed below will be modified with the remaining attributes -->
+          <!-- If the attribute already existed, it will be overwritten -->
+          <!-- Note that the type and name elements are required -->
+          <modify_element type="joint" name="gripper_outer_finger_left_joint" actuatorfrcrange="-8 8"/>
+          <modify_element type="joint" name="gripper_outer_finger_right_joint" actuatorfrcrange="-8 8"/>
+          <modify_element type="joint" name="gripper_inner_finger_left_joint" actuatorfrcrange="-8 8"/>
+          <modify_element type="joint" name="gripper_finger_right_joint" actuatorfrcrange="-8 8"/>
+          <modify_element type="joint" name="gripper_fingertip_left_joint" actuatorfrcrange="-8 8"/>
+          <modify_element type="joint" name="gripper_fingertip_right_joint" actuatorfrcrange="-8 8"/>
+          <modify_element type="joint" name="gripper_finger_joint" actuatorfrcrange="-8 8" damping="1.5"/>
+      </processed_inputs>
+    </mujoco_inputs>
+  </xacro:macro>
 </robot>

Commit message: add sim_type arg for the ros2-control tags

File: pal_pro_gripper_description/robots/pal_pro_gripper.urdf.xacro (robot description, xacro)
@@ -51,4 +51,6 @@
     </xacro:if>
     <!-- ROS 2 Control -->
-    <xacro:pal_pro_gripper_ros2_control use_sim_time="${use_sim_time}" sim_type="${sim_type}" />
+    <xacro:if value="${sim_type != 'mujoco'}">
+        <xacro:pal_pro_gripper_ros2_control use_sim_time="${use_sim_time}" sim_type="${sim_type}"/>
+    </xacro:if>
 </robot>

File: pal_pro_gripper_description/ros2_control/ros2_control.urdf.xacro (robot description, xacro)
@@ -13,5 +13,5 @@
  -->
 <robot xmlns:xacro="http://ros.org/wiki/xacro" name="pal_pro_gripper">
-  <xacro:macro name="pal_pro_gripper_ros2_control" params="use_sim_time:=^|false">
+  <xacro:macro name="pal_pro_gripper_ros2_control" params="use_sim_time:=^|false sim_type:=^|gazebo">
     <xacro:include filename="$(find pal_pro_gripper_description)/urdf/gripper.ros2_control.xacro" />
     <ros2_control name="ros2_control_pal_pro_gripper_system" type="system">

File: pal_pro_gripper_description/urdf/gripper.ros2_control.xacro (robot description, xacro)
@@ -13,5 +13,5 @@
 -->
 <robot xmlns:xacro="http://ros.org/wiki/xacro">
-  <xacro:macro name="ros2_control_pal_pro_gripper" params="name reduction sim_type:=gazebo">
+  <xacro:macro name="ros2_control_pal_pro_gripper" params="name reduction sim_type:=^|gazebo">
     <xacro:macro name="ros2_control_pal_pro_gripper_mimic_joint" params="mimic_joint_name actuated_joint_name multiplier ">
       <joint name="${mimic_joint_name}">
