Commit message: align to the new mujoco_ros2_control

File: pal_pro_gripper_description/mujoco/mj_tags.xacro (robot description, xacro)
@@ -3,5 +3,5 @@
     <xacro:macro name="mj_gripper_actuators" params="name">
         <xacro:if value="${mj_control == 'position' or mj_control == 'motor'}">
-            <position name="${name}_position" joint="${name}_inner_finger_left_joint" kp="100" ctrlrange=" 0 0.802851 " />
+            <position name="${name}_finger_joint" joint="${name}_finger_joint" kp="100" ctrlrange=" 0 0.07938 " />
         </xacro:if>
     </xacro:macro>
@@ -15,5 +15,11 @@
         <connect name="${name}_r" body1="${name}_fingertip_right_link" body2="${name}_outer_finger_right_link"  active="true" anchor="${anchor_r}" solref="0.005 1" solimp="0.95 0.99 0.001"/>
         <connect name="${name}_l" body1="${name}_fingertip_left_link" body2="${name}_outer_finger_left_link" active="true"  anchor="${anchor_l}" solref="0.005 1" solimp="0.95 0.99 0.001"/>
-        <joint joint1="${name}_inner_finger_left_joint" joint2="${name}_inner_finger_right_joint" polycoef="0 1 0 0 0" solref="0.005 1" solimp="0.95 0.99 0.001"/>
+        <joint joint1="${name}_finger_joint" joint2="${name}_outer_finger_right_joint" polycoef="0 -0.1208  0 0 0" solref="0.005 1" solimp="0.95 0.99 0.001"/>
+        <joint joint1="${name}_finger_joint" joint2="${name}_inner_finger_right_joint" polycoef="0 -0.1208  0 0 0" solref="0.005 1" solimp="0.95 0.99 0.001"/>
+        <joint joint1="${name}_finger_joint" joint2="${name}_fingertip_right_joint"    polycoef="0 0.1208  0 0 0"  solref="0.005 1" solimp="0.95 0.99 0.001"/>
+        <joint joint1="${name}_finger_joint" joint2="${name}_finger_right_joint"       polycoef="0 4.545 0 0 0"  solref="0.005 1" solimp="0.95 0.99 0.001"/>
+        <joint joint1="${name}_finger_joint" joint2="${name}_outer_finger_left_joint"  polycoef="0 -0.1208  0 0 0" solref="0.005 1" solimp="0.95 0.99 0.001"/>
+        <joint joint1="${name}_finger_joint" joint2="${name}_inner_finger_left_joint"  polycoef="0 -0.1208  0 0 0" solref="0.005 1" solimp="0.95 0.99 0.001"/>
+        <joint joint1="${name}_finger_joint" joint2="${name}_fingertip_left_joint"     polycoef="0 0.1208  0 0 0"  solref="0.005 1" solimp="0.95 0.99 0.001"/>
     </xacro:macro>
     <xacro:macro name="mj_gripper_actuator_pose" params="property_name">

File: pal_pro_gripper_description/robots/pal_pro_gripper.urdf.xacro (robot description, xacro)
@@ -11,5 +11,5 @@
      <!-- Mujoco args -->
     <xacro:arg name="sim_type" default="gazebo" />
-    <xacro:arg name="mj_control" default="false" />
+    <xacro:arg name="mj_control" default="position" />
     <xacro:arg name="world_name" default="floor" />
     <!-- PROPERTIES -->
@@ -37,22 +37,62 @@
         <origin xyz="0.0 0.0 0.08" rpy="0 0 0" />
     </xacro:pal_pro_gripper>
+    <!-- MUJOCO -->
     <xacro:if value="${sim_type == 'mujoco' or sim_type == 'mujoco-ros2-control'}">
-        <!-- MUJOCO -->
+        <!-- Mujoco Includes -->
         <xacro:include filename="$(find pal_pro_gripper_description)/mujoco/mj_tags.xacro" />
         <xacro:include filename="$(find pal_mujoco_scenes)/scenes/${world_name}.xacro" />
-        <mujoco>
+        <mujoco_inputs>
             <!-- Mujoco environment -->
-            <xacro:mj_common light_target="base_link"/>
-            <!-- Contact-->
-            <xacro:mj_gripper_contact name="gripper"/>
-            <!-- Actuator-->
-            <xacro:if value="${sim_type == 'mujoco'}">
-                <!-- Equality-->
-                <xacro:mj_gripper_equality name="gripper" anchor_r="0.014 -0.0015 0" anchor_l="0.014 -0.001 0"/>
-                <actuator>
-                    <xacro:mj_gripper_actuators name="gripper"/>
-                </actuator>
-            </xacro:if>
-        </mujoco>
+            <!-- <xacro:mj_common light_target="base_link"/> -->
+            <!-- Mujoco environment -->
+            <scene>
+                <xacro:mj_scene/>
+            </scene>
+            <raw_inputs>
+                <!-- Contact-->
+                <xacro:mj_gripper_contact name="gripper"/>
+                <!-- Actuator-->
+                <xacro:if value="${sim_type == 'mujoco' or sim_type == 'mujoco-ros2-control'}">
+                    <!-- Equality-->
+                    <xacro:mj_gripper_equality name="gripper" anchor_r="0.014 -0.0015 0" anchor_l="0.014 -0.001 0"/>
+                    <actuator>
+                        <xacro:mj_gripper_actuators name="gripper"/>
+                    </actuator>
+                </xacro:if>
+                <default>
+                    <default class="visual">
+                        <geom group="2" type="mesh" contype="0" conaffinity="0"/>
+                    </default>
+                    <default class="collision">
+                        <geom group="3" type="mesh"/>
+                    </default>
+                </default>
+            </raw_inputs>
+            <processed_inputs>
+                <!-- Specifying decompose_mesh will set the `decompose` flag when using obj2mjcf -->
+                <!-- <decompose_mesh mesh_name="arm2_link" threshold="0.05"/>
+                <decompose_mesh mesh_name="arm3_link" threshold="0.05"/> -->
+                <!-- <decompose_mesh mesh_name="arm4_link" threshold="0.05"/> -->
+                <!-- The camera with the specified values will be added at the specified site name. -->
+                <!-- The position and quaterinion will be filled in by the converter -->
+                <!-- <camera site="pelvis_1_link" name="camera" fovy="58" mode="fixed" resolution="640 480" pos="2 2 2" quat="1 0 0 0"/> -->
+                <!-- Adds a lidar tag below a site tag to support a lidar sensor. -->
+                <!-- In the URDF, we assume that that the sensor frame has the Z-axis pointed directly up in the sensor -->
+                <!-- frame. This tag will create rangefinders in the MJCF between min_angle and max_angle at each -->
+                <!-- angle_increment rotated about the replicate frame's Y axis. The hardware intercface then combines -->
+                <!-- them into a single LaserScan message. -->
+                <!-- <lidar ref_site="torso_link" sensor_name="rf" min_angle="-0.3" max_angle="0.3" angle_increment="0.025" /> -->
+                <!-- The element with the type and name as listed below will be modified with the remaining attributes -->
+                <!-- If the attribute already existed, it will be overwritten -->
+                <!-- Note that the type and name elements are required -->
+                <modify_element type="joint" name="gripper_outer_finger_left_joint" actuatorfrcrange="-8 8"/>
+                <modify_element type="joint" name="gripper_outer_finger_right_joint" actuatorfrcrange="-8 8"/>
+                <modify_element type="joint" name="gripper_inner_finger_left_joint" actuatorfrcrange="-8 8"/>
+                <modify_element type="joint" name="gripper_finger_right_joint" actuatorfrcrange="-8 8"/>
+                <modify_element type="joint" name="gripper_fingertip_left_joint" actuatorfrcrange="-8 8"/>
+                <modify_element type="joint" name="gripper_fingertip_right_joint" actuatorfrcrange="-8 8"/>
+                <modify_element type="joint" name="gripper_finger_joint" actuatorfrcrange="-8 8" damping="1.5"/>
+            </processed_inputs>
+        </mujoco_inputs>
     </xacro:if>
     <!-- ROS 2 Control -->

File: pal_pro_gripper_description/ros2_control/ros2_control.urdf.xacro (robot description, xacro)
@@ -13,5 +13,5 @@
  -->
 <robot xmlns:xacro="http://ros.org/wiki/xacro" name="pal_pro_gripper">
-  <xacro:macro name="pal_pro_gripper_ros2_control" params="use_sim_time:=^|false sim_type:=no-simulation">
+  <xacro:macro name="pal_pro_gripper_ros2_control" params="use_sim_time:=^|false">
     <xacro:include filename="$(find pal_pro_gripper_description)/urdf/gripper.ros2_control.xacro" />
     <ros2_control name="ros2_control_pal_pro_gripper_system" type="system">
@@ -19,5 +19,7 @@
         <xacro:if value="$(arg use_sim_time)">
           <xacro:if value="${sim_type == 'mujoco-ros2-control'}">
-            <plugin>mujoco_ros2_control/MujocoSystem</plugin>
+            <plugin>mujoco_ros2_control/MujocoSystemInterface</plugin>
+            <!-- Override the slowdown settings in the Simulate App and run at 3x speed -->
+            <param name="sim_speed_factor">1.0</param>
           </xacro:if>
           <xacro:if value="${sim_type == 'gazebo'}">
@@ -35,5 +37,5 @@
       </hardware>
       <!-- pal-pro-gripper -->
-      <xacro:ros2_control_pal_pro_gripper name="gripper" reduction="1.0"  sim_type="${sim_type}"/>
+      <xacro:ros2_control_pal_pro_gripper name="gripper" reduction="1.0"/>
     </ros2_control>
   </xacro:macro>

File: pal_pro_gripper_description/urdf/gripper.ros2_control.xacro (robot description, xacro)
@@ -13,6 +13,6 @@
 -->
 <robot xmlns:xacro="http://ros.org/wiki/xacro">
-  <xacro:macro name="ros2_control_pal_pro_gripper" params="name reduction sim_type:=no-simulation">
-    <xacro:macro name="ros2_control_pal_pro_gripper_mimic_joint" params="mimic_joint_name actuated_joint_name multiplier sim_type:=no-simulation">
+  <xacro:macro name="ros2_control_pal_pro_gripper" params="name reduction">
+    <xacro:macro name="ros2_control_pal_pro_gripper_mimic_joint" params="mimic_joint_name actuated_joint_name multiplier">
       <joint name="${mimic_joint_name}">
         <param name="mimic">${actuated_joint_name}</param>

Commit message: parametrize common args in gripper_limits.xacro

File: pal_pro_gripper_description/mujoco/mj_tags.xacro (robot description, xacro)
@@ -1,10 +1,11 @@
 <?xml version="1.0"?>
-<robot xmlns:xacro="http://ros.org/wiki/xacro" name="pal_pro_gripper">
-    <xacro:macro name="mj_gripper_actuators" params="name">
+<robot xmlns:xacro="http://ros.org/wiki/xacro">
+    <xacro:macro name="mj_gripper_actuators" params="name mj_control">
+        <xacro:include filename="$(find pal_pro_gripper_description)/urdf/gripper_limits.xacro" />
         <xacro:if value="${mj_control == 'position'}">
-            <position name="${name}_finger_joint_position" joint="${name}_finger_joint" kp="100" ctrlrange=" 0 0.07938 " />
+            <position name="${name}_finger_joint_position" joint="${name}_finger_joint" kp="100" ctrlrange="${finger_lower_limit} ${finger_upper_limit}" />
         </xacro:if>
         <xacro:if value="${mj_control == 'motor'}">
-            <motor name="${name}_finger_joint_motor" joint="${name}_finger_joint"  ctrllimited="true" ctrlrange="-8 8" />
+            <motor name="${name}_finger_joint_motor" joint="${name}_finger_joint"  ctrllimited="true" ctrlrange="${finger_mj_min_effort} ${finger_mj_max_effort}" />
         </xacro:if>
     </xacro:macro>
@@ -16,13 +17,14 @@
     </xacro:macro>
     <xacro:macro name="mj_gripper_equality" params="name anchor_r anchor_l" >
+        <xacro:include filename="$(find pal_pro_gripper_description)/urdf/gripper_limits.xacro" />
         <connect name="${name}_r" body1="${name}_fingertip_right_link" body2="${name}_outer_finger_right_link"  active="true" anchor="${anchor_r}" solref="0.005 1" solimp="0.95 0.99 0.001"/>
         <connect name="${name}_l" body1="${name}_fingertip_left_link" body2="${name}_outer_finger_left_link" active="true"  anchor="${anchor_l}" solref="0.005 1" solimp="0.95 0.99 0.001"/>
-        <joint joint1="${name}_finger_joint" joint2="${name}_outer_finger_right_joint" polycoef="0 -0.1208  0 0 0" solref="0.005 1" solimp="0.95 0.99 0.001"/>
-        <joint joint1="${name}_finger_joint" joint2="${name}_inner_finger_right_joint" polycoef="0 -0.1208  0 0 0" solref="0.005 1" solimp="0.95 0.99 0.001"/>
-        <joint joint1="${name}_finger_joint" joint2="${name}_fingertip_right_joint"    polycoef="0 0.1208  0 0 0"  solref="0.005 1" solimp="0.95 0.99 0.001"/>
-        <joint joint1="${name}_finger_joint" joint2="${name}_finger_right_joint"       polycoef="0 4.545 0 0 0"  solref="0.005 1" solimp="0.95 0.99 0.001"/>
-        <joint joint1="${name}_finger_joint" joint2="${name}_outer_finger_left_joint"  polycoef="0 -0.1208  0 0 0" solref="0.005 1" solimp="0.95 0.99 0.001"/>
-        <joint joint1="${name}_finger_joint" joint2="${name}_inner_finger_left_joint"  polycoef="0 -0.1208  0 0 0" solref="0.005 1" solimp="0.95 0.99 0.001"/>
-        <joint joint1="${name}_finger_joint" joint2="${name}_fingertip_left_joint"     polycoef="0 0.1208  0 0 0"  solref="0.005 1" solimp="0.95 0.99 0.001"/>
+        <joint joint1="${name}_finger_joint" joint2="${name}_outer_finger_right_joint" polycoef="0 ${1.0 / outer_finger_multiplier}  0 0 0" solref="0.005 1" solimp="0.95 0.99 0.001"/>
+        <joint joint1="${name}_finger_joint" joint2="${name}_inner_finger_right_joint" polycoef="0 ${1.0 / inner_finger_multiplier}  0 0 0" solref="0.005 1" solimp="0.95 0.99 0.001"/>
+        <joint joint1="${name}_finger_joint" joint2="${name}_fingertip_right_joint"    polycoef="0 ${1.0 / fingertip_multiplier}  0 0 0"  solref="0.005 1" solimp="0.95 0.99 0.001"/>
+        <joint joint1="${name}_finger_joint" joint2="${name}_finger_right_joint"       polycoef="0 ${1.0 / finger_right_joint_multiplier} 0 0 0"  solref="0.005 1" solimp="0.95 0.99 0.001"/>
+        <joint joint1="${name}_finger_joint" joint2="${name}_outer_finger_left_joint"  polycoef="0 ${1.0 / outer_finger_multiplier}  0 0 0" solref="0.005 1" solimp="0.95 0.99 0.001"/>
+        <joint joint1="${name}_finger_joint" joint2="${name}_inner_finger_left_joint"  polycoef="0 ${1.0 / inner_finger_multiplier}  0 0 0" solref="0.005 1" solimp="0.95 0.99 0.001"/>
+        <joint joint1="${name}_finger_joint" joint2="${name}_fingertip_left_joint"     polycoef="0 ${1.0 / fingertip_multiplier}  0 0 0"  solref="0.005 1" solimp="0.95 0.99 0.001"/>
     </xacro:macro>
     <xacro:macro name="mj_gripper_actuator_pose" params="property_name">

File: pal_pro_gripper_description/urdf/gripper.urdf.xacro (robot description, xacro)
@@ -3,4 +3,5 @@
   <!-- A finger of the pal_pro_gripper -->
   <xacro:macro name="pro_finger" params="name side reflect finger_offset:=0">
+    <xacro:include filename="$(find pal_pro_gripper_description)/urdf/gripper_limits.xacro" />
     <!-- Screw link -->
     <link name="${name}_screw_${side}_link">
@@ -21,5 +22,5 @@
       <child link="${name}_screw_${side}_link"/>
       <axis xyz="0 1 0"/>
-      <limit lower="${gripper_lower_limit}" upper="0.07" velocity="2" effort="10.0"/>
+      <limit lower="${gripper_lower_limit}" upper="${finger_upper_limit}" velocity="2" effort="10.0"/>
       <safety_controller k_position="20" k_velocity="20" soft_lower_limit="${gripper_lower_limit + gripper_eps}" soft_upper_limit="${0.07 - gripper_eps}" />
       <xacro:if value="${side == 'left'}">
@@ -27,5 +28,5 @@
       </xacro:if>
       <xacro:unless value="${side == 'left'}">
-        <mimic joint="${name}_finger_joint" multiplier="0.22" offset="0" />
+        <mimic joint="${name}_finger_joint" multiplier="${finger_right_joint_multiplier}" offset="0" />
       </xacro:unless>
     </joint>
@@ -79,5 +80,5 @@
       <axis xyz="0 0 1"/>
       <limit lower="${-42.840* deg_to_rad}" upper="${8.001 * deg_to_rad}" velocity="2" effort="0.1"/>
-      <mimic joint="${name}_finger_joint" multiplier="-8.28" offset="0.0"/>
+      <mimic joint="${name}_finger_joint" multiplier="${inner_finger_multiplier}" offset="0.0"/>
     </joint>
     <!-- Outer finger -->
@@ -106,5 +107,5 @@
       <axis xyz="0 0 1"/>
       <limit lower="${-42.840 * deg_to_rad}" upper="${8.001 * deg_to_rad}" velocity="2" effort="0.1"/>
-      <mimic joint="${name}_finger_joint" multiplier="-8.28" offset="0.0"/>
+      <mimic joint="${name}_finger_joint" multiplier="${outer_finger_multiplier}" offset="0.0"/>
     </joint>
     <!-- Fingertip -->
@@ -133,5 +134,5 @@
       <axis xyz="0 0 1"/>
       <limit lower="${-8.001 * deg_to_rad}" upper="${42.840 * deg_to_rad}" velocity="2" effort="0.1"/>
-      <mimic joint="${name}_finger_joint" multiplier="8.28" offset="0.0"/>
+      <mimic joint="${name}_finger_joint" multiplier="${fingertip_multiplier}" offset="0.0"/>
     </joint>
   </xacro:macro>

Commit message: Add MuJoCo tag properties for mujoco simulation

File: pal_pro_gripper_description/mujoco/mj_tags.xacro (robot description, xacro)
@@ -17,3 +17,9 @@
         <joint joint1="${name}_inner_finger_left_joint" joint2="${name}_inner_finger_right_joint" polycoef="0 1 0 0 0" solref="0.005 1" solimp="0.95 0.99 0.001"/>
     </xacro:macro>
+    <xacro:macro name="mj_gripper_actuator_pose" params="property_name">
+        <xacro:property name="${property_name}" value="0" scope="parent"/>
+    </xacro:macro>
+    <xacro:macro name="mj_gripper_pose" params="property_name">
+        <xacro:property name="${property_name}" value="0 0 0 0 0 0 0 0" scope="parent"/>
+    </xacro:macro>
 </robot>
